File: Eagle PCBs/Slave.brd (EAGLE design)
At the start: 46.7 x 104.1 mm, 24 parts, among them Q1 TIP120

Commit message: Changed TIP120 resistor value and added some WIP files
Parts:
- R1: value 2.2k -> 1K
Changed lines of the file:
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@@
 <attribute name="VALUE" x="30.353" y="41.91" size="1.778" layer="27" ratio="10"/>
 </element>
-<element name="R1" library="rcl" library_urn="urn:adsk.eagle:library:334" package="0207/10" package3d_urn="urn:adsk.eagle:package:23491/2" value="2.2k" x="21.59" y="77.978" smashed="yes">
+<element name="R1" library="rcl" library_urn="urn:adsk.eagle:library:334" package="0207/10" package3d_urn="urn:adsk.eagle:package:23491/2" value="1K" x="21.59" y="77.978" smashed="yes">
 <attribute name="NAME" x="18.542" y="79.502" size="1.27" layer="25" ratio="10"/>
 <attribute name="POPULARITY" value="81" x="54.61" y="3.048" size="1.778" layer="27" display="off"/>
