File: Eagle PCBs/Slave.sch (EAGLE design)
At the start: 25 parts, among them Q1 TIP120

Commit message: Slave PCB WIP
Parts:
- removed LED_PWM: Header, pinhead:PINHD-1X1
Connections:
- removed net DIMMER_PWM_PIN: LED_PWM.1, R1.1
- new net NANO_1_DIM: NANO-1-6.S, R1.1
Other:
- moved on the sheet: LED_STRIP, Q1, R1
Changed lines of the file:
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@@
 <part name="Q1" library="transistor-power" library_urn="urn:adsk.eagle:library:400" deviceset="TIP120" device="" package3d_urn="urn:adsk.eagle:package:29488/1"/>
 <part name="LED_STRIP" library="SamacSys_Parts" deviceset="215760-3002" device=""/>
-<part name="LED_PWM" library="pinhead" library_urn="urn:adsk.eagle:library:325" deviceset="PINHD-1X1" device="" package3d_urn="urn:adsk.eagle:package:22485/2" value="Header"/>
 <part name="RS485-SLAVE-1" library="A10 Library" deviceset="MAX487CPA" device="" package3d_urn="urn:adsk.eagle:package:29519/2"/>
 <part name="NANO-1" library="con-molex" library_urn="urn:adsk.eagle:library:165" deviceset="22-23-2061" device="" package3d_urn="urn:adsk.eagle:package:8078637/1" value="6P"/>
@@
 </plain>
 <instances>
-<instance part="R1" gate="G$1" x="10.16" y="43.18" smashed="yes" rot="R270">
-<attribute name="NAME" x="11.6586" y="46.99" size="1.778" layer="95" rot="R270"/>
-<attribute name="VALUE" x="6.858" y="46.99" size="1.778" layer="96" rot="R270"/>
-</instance>
-<instance part="Q1" gate="1" x="17.78" y="20.32" smashed="yes">
-<attribute name="NAME" x="22.86" y="22.86" size="1.778" layer="95"/>
-<attribute name="VALUE" x="22.86" y="20.32" size="1.778" layer="96"/>
-</instance>
-<instance part="LED_STRIP" gate="G$1" x="25.4" y="33.02" smashed="yes" rot="R90">
-<attribute name="NAME" x="17.78" y="49.53" size="1.778" layer="95" rot="R90" align="center-left"/>
-<attribute name="VALUE" x="20.32" y="49.53" size="1.778" layer="96" rot="R90" align="center-left"/>
-</instance>
-<instance part="LED_PWM" gate="G$1" x="29.464" y="71.12" smashed="yes">
-<attribute name="NAME" x="23.114" y="74.295" size="1.778" layer="95"/>
-<attribute name="VALUE" x="23.114" y="66.04" size="1.778" layer="96"/>
+<instance part="R1" gate="G$1" x="10.16" y="48.26" smashed="yes" rot="R270">
+<attribute name="NAME" x="11.6586" y="52.07" size="1.778" layer="95" rot="R270"/>
+<attribute name="VALUE" x="6.858" y="52.07" size="1.778" layer="96" rot="R270"/>
+</instance>
+<instance part="Q1" gate="1" x="17.78" y="25.4" smashed="yes">
+<attribute name="NAME" x="22.86" y="27.94" size="1.778" layer="95"/>
+<attribute name="VALUE" x="22.86" y="25.4" size="1.778" layer="96"/>
+</instance>
+<instance part="LED_STRIP" gate="G$1" x="25.4" y="38.1" smashed="yes" rot="R90">
+<attribute name="NAME" x="17.78" y="54.61" size="1.778" layer="95" rot="R90" align="center-left"/>
+<attribute name="VALUE" x="20.32" y="54.61" size="1.778" layer="96" rot="R90" align="center-left"/>
 </instance>
 <instance part="RS485-SLAVE-1" gate="G$1" x="160.02" y="55.88" smashed="yes">
@@
 <segment>
 <pinref part="Q1" gate="1" pin="E"/>
-<wire x1="20.32" y1="15.24" x2="20.32" y2="5.08" width="0.1524" layer="91"/>
-<label x="20.32" y="5.08" size="1.778" layer="95" rot="R90"/>
+<wire x1="20.32" y1="20.32" x2="20.32" y2="10.16" width="0.1524" layer="91"/>
+<label x="20.32" y="10.16" size="1.778" layer="95" rot="R90"/>
 </segment>
 <segment>
@@
 </segment>
 </net>
-<net name="DIMMER_PWM_PIN" class="0">
-<segment>
-<pinref part="R1" gate="G$1" pin="1"/>
-<wire x1="10.16" y1="48.26" x2="10.16" y2="71.12" width="0.1524" layer="91"/>
-<label x="10.16" y="48.26" size="1.778" layer="95" rot="R90"/>
-<pinref part="LED_PWM" gate="G$1" pin="1"/>
-<wire x1="10.16" y1="71.12" x2="26.924" y2="71.12" width="0.1524" layer="91"/>
-</segment>
-</net>
 <net name="N$1" class="0">
 <segment>
 <pinref part="R1" gate="G$1" pin="2"/>
-<wire x1="10.16" y1="38.1" x2="10.16" y2="20.32" width="0.1524" layer="91"/>
+<wire x1="10.16" y1="43.18" x2="10.16" y2="25.4" width="0.1524" layer="91"/>
 <pinref part="Q1" gate="1" pin="B"/>
-<wire x1="10.16" y1="20.32" x2="15.24" y2="20.32" width="0.1524" layer="91"/>
+<wire x1="10.16" y1="25.4" x2="15.24" y2="25.4" width="0.1524" layer="91"/>
 </segment>
 </net>
@@
 <segment>
 <pinref part="Q1" gate="1" pin="C"/>
-<wire x1="20.32" y1="25.4" x2="20.32" y2="33.02" width="0.1524" layer="91"/>
+<wire x1="20.32" y1="30.48" x2="20.32" y2="38.1" width="0.1524" layer="91"/>
 <pinref part="LED_STRIP" gate="G$1" pin="2"/>
-<wire x1="20.32" y1="33.02" x2="25.4" y2="33.02" width="0.1524" layer="91"/>
-<label x="20.32" y="33.02" size="1.778" layer="95" rot="R90"/>
+<wire x1="20.32" y1="38.1" x2="25.4" y2="38.1" width="0.1524" layer="91"/>
+<label x="20.32" y="38.1" size="1.778" layer="95" rot="R90"/>
 </segment>
 </net>
@@
 <segment>
 <pinref part="LED_STRIP" gate="G$1" pin="1"/>
-<wire x1="27.94" y1="33.02" x2="38.1" y2="33.02" width="0.1524" layer="91"/>
-<label x="33.02" y="33.02" size="1.778" layer="95"/>
+<wire x1="27.94" y1="38.1" x2="38.1" y2="38.1" width="0.1524" layer="91"/>
+<label x="33.02" y="38.1" size="1.778" layer="95"/>
 </segment>
 </net>
@@
 </segment>
 </net>
+<net name="NANO_1_DIM" class="0">
+<segment>
+<pinref part="R1" gate="G$1" pin="1"/>
+<wire x1="10.16" y1="53.34" x2="10.16" y2="71.12" width="0.1524" layer="91"/>
+<label x="10.16" y="55.88" size="1.778" layer="95" rot="R90"/>
+</segment>
+<segment>
+<pinref part="NANO-1" gate="-6" pin="S"/>
+<wire x1="157.48" y1="12.7" x2="149.86" y2="12.7" width="0.1524" layer="91"/>
+<label x="142.24" y="10.16" size="1.778" layer="95"/>
+</segment>
+</net>

Commit message: Changed TIP120 resistor value and added some WIP files
Parts:
- R1: value 2.2k -> 1K
Changed lines of the file:
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@@
 </classes>
 <parts>
-<part name="R1" library="rcl" library_urn="urn:adsk.eagle:library:334" deviceset="R-EU_" device="0207/10" package3d_urn="urn:adsk.eagle:package:23491/2" value="2.2k"/>
+<part name="R1" library="rcl" library_urn="urn:adsk.eagle:library:334" deviceset="R-EU_" device="0207/10" package3d_urn="urn:adsk.eagle:package:23491/2" value="1K"/>
 <part name="Q1" library="transistor-power" library_urn="urn:adsk.eagle:library:400" deviceset="TIP120" device="" package3d_urn="urn:adsk.eagle:package:29488/1"/>
 <part name="LED_STRIP" library="SamacSys_Parts" deviceset="215760-3002" device=""/>
